Commit message: Minor changes to the controllers for the hybrid MPC benchmark.
Minor changes to the controllers for the hybrid MPC benchmark.

File: examples/cart_pole.urdf (robot description, URDF)
Before this commit: robot CartPole, 3 links, 2 joints
Links:
- added link wall; collision box size=.2 0 4.1; visual box size=.2 0 4.1
- link ground: geometry visual box size=6 0 .5
- link pole: geometry collision sphere radius=.05; visual cylinder length=2 radius=.05
